File: eagle/power_v2.brd (EAGLE design)
At the start: 98.7 x 50.8 mm, 14 parts, among them X1 736880-49, X2 736880-49, X3 736880-49, X4 736880-49, X5 736880-49

Commit message: cinch -> svorkovnice
Parts:
- removed X1, X2, X3, X4, X5: 736880-49, con-conrad:736880-49
- added GND&1, GND&2, GND&3, GND&4, GND&5, VCC, VCC1, VCC2, VCC3, VCC4: WIREPAD3,17/1,3, wirepad:3,17/1,3
Connections:
- new net N$1: GND&1.1
- net GND: now also GND&2.1, GND&3.1, GND&4.1, GND&5.1; no longer X1.2, X2.2, X3.2, X4.2, X5.2
- net N$6: now also VCC.1, VCC1.1, VCC2.1, VCC3.1, VCC4.1; no longer X1.1, X2.1, X3.1, X4.1, X5.1
Routing:
- net N$6: track 216.9 -> 206.3 mm
Changed lines of the file:
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@@
 <setting verticaltext="up"/>
 </settings>
-<grid distance="1.27" unitdist="mm" unit="mm" style="lines" multiple="1" display="yes" altdistance="0.635" altunitdist="mm" altunit="mm"/>
+<grid distance="2.54" unitdist="mm" unit="mm" style="lines" multiple="1" display="yes" altdistance="0.635" altunitdist="mm" altunit="mm"/>
 <layers>
 <layer number="1" name="Top" color="4" fill="1" visible="yes" active="yes"/>
@@
 <hole x="5.08" y="43.18" drill="4"/>
 <hole x="93.98" y="43.18" drill="4"/>
-<hole x="19.05" y="2.54" drill="4"/>
-<hole x="80.01" y="2.54" drill="4"/>
+<hole x="20.32" y="12.7" drill="4"/>
+<hole x="78.74" y="12.7" drill="4"/>
 <text x="36.83" y="36.83" size="1.778" layer="16" font="vector" rot="MR0">ledbar power board</text>
 </plain>
@@
 <element name="+5V" library="wirepad" package="4,16O1,6" value="WIREPAD4,16O1,6" x="54.61" y="36.83"/>
 <element name="GND" library="wirepad" package="4,16O1,6" value="WIREPAD4,16O1,6" x="44.45" y="36.83"/>
-<element name="X1" library="con-conrad" package="736880-49" value="736880-49" x="49.53" y="6.35" rot="R90"/>
 <element name="LED1" library="led" package="LED5MM" value="" x="77.47" y="36.83"/>
 <element name="R1" library="resistor" package="R1206" value="200R" x="69.85" y="36.83" rot="MR0"/>
 <element name="C1" library="resistor" package="E5-10,5" value="1000u" x="92.71" y="21.59"/>
-<element name="X2" library="con-conrad" package="736880-49" value="736880-49" x="90.17" y="6.35" rot="R90"/>
 <element name="C2" library="resistor" package="E5-10,5" value="1000u" x="72.39" y="21.59"/>
-<element name="X3" library="con-conrad" package="736880-49" value="736880-49" x="29.21" y="6.35" rot="R90"/>
 <element name="C3" library="resistor" package="E5-10,5" value="1000u" x="52.07" y="21.59"/>
-<element name="X4" library="con-conrad" package="736880-49" value="736880-49" x="69.85" y="6.35" rot="R90"/>
 <element name="C4" library="resistor" package="E5-10,5" value="1000u" x="11.43" y="21.59"/>
-<element name="X5" library="con-conrad" package="736880-49" value="736880-49" x="8.89" y="6.35" rot="R90"/>
 <element name="C5" library="resistor" package="E5-10,5" value="1000u" x="31.75" y="21.59"/>
+<element name="GND&amp;1" library="wirepad" package="3,17/1,3" value="WIREPAD3,17/1,3" x="12.7" y="5.08"/>
+<element name="VCC" library="wirepad" package="3,17/1,3" value="WIREPAD3,17/1,3" x="7.62" y="5.08"/>
+<element name="GND&amp;2" library="wirepad" package="3,17/1,3" value="WIREPAD3,17/1,3" x="33.02" y="5.08"/>
+<element name="VCC1" library="wirepad" package="3,17/1,3" value="WIREPAD3,17/1,3" x="27.94" y="5.08"/>
+<element name="GND&amp;3" library="wirepad" package="3,17/1,3" value="WIREPAD3,17/1,3" x="53.34" y="5.08"/>
+<element name="VCC2" library="wirepad" package="3,17/1,3" value="WIREPAD3,17/1,3" x="48.26" y="5.08"/>
+<element name="GND&amp;4" library="wirepad" package="3,17/1,3" value="WIREPAD3,17/1,3" x="73.66" y="5.08"/>
+<element name="VCC3" library="wirepad" package="3,17/1,3" value="WIREPAD3,17/1,3" x="68.58" y="5.08"/>
+<element name="GND&amp;5" library="wirepad" package="3,17/1,3" value="WIREPAD3,17/1,3" x="93.98" y="5.08"/>
+<element name="VCC4" library="wirepad" package="3,17/1,3" value="WIREPAD3,17/1,3" x="88.9" y="5.08"/>
 </elements>
 <signals>
 <signal name="N$6">
 <contactref element="C3" pad="+"/>
-<contactref element="X3" pad="1"/>
 <contactref element="C4" pad="+"/>
-<contactref element="X4" pad="1"/>
 <contactref element="C1" pad="+"/>
-<contactref element="X1" pad="1"/>
 <contactref element="+5V" pad="1"/>
 <contactref element="C2" pad="+"/>
-<contactref element="X2" pad="1"/>
 <contactref element="C5" pad="+"/>
-<contactref element="X5" pad="1"/>
 <contactref element="R1" pad="2"/>
-<wire x1="8.89" y1="21.59" x2="8.89" y2="2.43" width="1.27" layer="16"/>
-<wire x1="29.21" y1="21.59" x2="29.21" y2="2.43" width="1.27" layer="16"/>
-<wire x1="49.53" y1="21.59" x2="49.53" y2="2.43" width="1.27" layer="16"/>
-<wire x1="69.85" y1="21.59" x2="69.85" y2="2.43" width="1.27" layer="16"/>
-<wire x1="90.17" y1="21.59" x2="90.17" y2="2.43" width="1.27" layer="16"/>
 <wire x1="8.89" y1="21.59" x2="12.7" y2="25.4" width="1.27" layer="16"/>
 <wire x1="12.7" y1="25.4" x2="29.21" y2="25.4" width="1.27" layer="16"/>
@@
 <wire x1="54.61" y1="36.83" x2="54.61" y2="25.4" width="1.27" layer="16"/>
 <wire x1="68.428" y1="36.83" x2="54.61" y2="36.83" width="0.4064" layer="16"/>
+<contactref element="VCC" pad="1"/>
+<contactref element="VCC1" pad="1"/>
+<contactref element="VCC2" pad="1"/>
+<contactref element="VCC3" pad="1"/>
+<contactref element="VCC4" pad="1"/>
+<wire x1="69.85" y1="21.59" x2="68.58" y2="20.32" width="1.016" layer="16"/>
+<wire x1="68.58" y1="20.32" x2="68.58" y2="5.08" width="1.016" layer="16"/>
+<wire x1="90.17" y1="21.59" x2="88.9" y2="20.32" width="1.016" layer="16"/>
+<wire x1="88.9" y1="20.32" x2="88.9" y2="5.08" width="1.016" layer="16"/>
+<wire x1="49.53" y1="21.59" x2="48.26" y2="20.32" width="1.016" layer="16"/>
+<wire x1="48.26" y1="20.32" x2="48.26" y2="5.08" width="1.016" layer="16"/>
+<wire x1="29.21" y1="21.59" x2="27.94" y2="20.32" width="1.016" layer="16"/>
+<wire x1="27.94" y1="20.32" x2="27.94" y2="5.08" width="1.016" layer="16"/>
+<wire x1="8.89" y1="21.59" x2="7.62" y2="20.32" width="1.016" layer="16"/>
+<wire x1="7.62" y1="20.32" x2="7.62" y2="5.08" width="1.016" layer="16"/>
 </signal>
 <signal name="N$2">
@@
 <vertex x="0" y="-5.08"/>
 </polygon>
-<contactref element="X1" pad="2"/>
 <contactref element="C1" pad="-"/>
-<contactref element="X2" pad="2"/>
 <contactref element="C2" pad="-"/>
-<contactref element="X3" pad="2"/>
 <contactref element="C3" pad="-"/>
-<contactref element="X4" pad="2"/>
 <contactref element="C4" pad="-"/>
-<contactref element="X5" pad="2"/>
 <contactref element="C5" pad="-"/>
 <contactref element="GND" pad="1"/>
 <contactref element="LED1" pad="K"/>
+<contactref element="GND&amp;2" pad="1"/>
+<contactref element="GND&amp;3" pad="1"/>
+<contactref element="GND&amp;4" pad="1"/>
+<contactref element="GND&amp;5" pad="1"/>
+</signal>
+<signal name="N$1">
+<contactref element="GND&amp;1" pad="1"/>
 </signal>
 </signals>
